Commit message: changed root link to base_link

File: velma_description/defs/torso_mobile.urdf.xacro (robot description, xacro)
@@ -4,5 +4,6 @@
                         xmlns:sensor="http://playerstage.sourceforge.net/gazebo/xmlschema/#sensor"
                         xmlns:xacro="http://www.ros.org/wiki/xacro">
-  <xacro:macro name="velma_torso" params="*origin">
+  <!-- <xacro:macro name="velma_torso" params="*origin"> -->
+    <xacro:macro name="velma_torso">
     <xacro:macro name="wheel_inertia" params="m r h">
       <inertia ixx="${m*(3*r*r+h*h)/12}" ixy="0" ixz="0" iyy="${m*r*r/2}" iyz="0" izz="${m*(3*r*r+h*h)/12}" />
@@ -18,5 +19,6 @@
         <wheelSeparation>0.76</wheelSeparation>
         <wheelDiameter>0.2032</wheelDiameter>
-        <robotBaseFrame>torso_base</robotBaseFrame>
+        <!-- <robotBaseFrame>torso_base</robotBaseFrame> -->
+        <robotBaseFrame>base_link</robotBaseFrame>
         <commandTopic>/cmd_vel</commandTopic>
         <publishOdometryTf>true</publishOdometryTf>
@@ -37,4 +39,12 @@
       </plugin>
     </gazebo>
+    <link name="base_link">
+      <origin xyz="-0.081 0 0.1225" rpy="0.0 0 0" />
+    </link>
+    <joint name="base_torso_joint" type="fixed">
+      <origin xyz="0 0 0" rpy="0 0 0"/>
+      <parent link="base_link"/>
+      <child link="torso_base"/>
+    </joint>
 <!--
     <joint name="torso_base_joint" type="planar">
@@ -67,5 +77,5 @@
         <geometry>
           <box size="0.907 0.75 0.15" />
-          <!-- <mesh filename="package://omnivelma/meshes/collider/base.dae" /> -->
+          <mesh filename="package://omnivelma/meshes/collider/base.dae" />
         </geometry>
       </collision>

File: velma_description/robots/velma.urdf.xacro (robot description, xacro)
@@ -289,4 +289,10 @@
       </sensor>
     </gazebo>
+<!--     <link name="base_link"/>
+    <joint name="base_torso_joint" type="fixed">
+      <origin xyz="0 0 0" rpy="0 0 0"/>
+      <parent name="base_link"/>
+      <child name="torso_base"/>
+    </joint> -->
     <monokl name="monokl_l" parent="torso_base">
       <origin xyz="0 0.3 0.256" rpy="0 0 0" />
@@ -300,5 +306,5 @@
   </xacro:if>
   <velma_torso>
-    <origin xyz="0 0 0" rpy="0 0 0"/>
+    <!-- <origin xyz="0 0 0" rpy="0 0 0"/> -->
   </velma_torso>
   <kuka_lwr_arm parent="torso_link0" name="right" right="1">
